File: motion-PIR-18650.sch (EAGLE design)
At the start: 17 parts, among them Q1 APM2014N, Q2 AP3310G, T1 BTA16-600, T2 BC547

Commit message: Add files via upload
Parts:
- added BOOST-UP: 5V, lex-library:POWER-BOOST-UP
- added D1, D2: BAS40, diode:BAS40
- added R5: 100k, resistor:R-EU_0204/2V
- added S1: MAN. LED, switch:RDT1034
- added S2: OFF LED, switch:RDT1034
- added U$2: POWER-BOOST-UP, lex-library:POWER-BOOST-UP
- LED1: value LED -> 1W
- R3: value 10R -> 2R
- R4: value 47k -> 100k
Connections:
- removed net N$12: Q2.D, R3.2
- new net LED: BOOST-UP.OUT+, D1.A, R3.2
- new net N$13: Q2.S, S2.B
- new net N$14: BOOST-UP.IN+, Q2.D
- new net SAFE++: D1.C, D2.C, PIR_SENSOR.1
- net GND: now also BOOST-UP.IN-, BOOST-UP.OUT-, R5.1, S1.A1
- net N$1: now also S1.B
- net PIR: now also R5.2
- net SAFE+: now also S2.A1; no longer PIR_SENSOR.1, Q2.S
- net VCC_5V: now also D2.A
Other:
- moved on the sheet: LED1, Q1, Q2, R3, R4

Commit message: Add files via upload
Parts:
- R3: value 2R -> 5R
Other:
- note added: "1. R3 can be replaced by driver NSI50350AST3G 350mA."
- note added: "2. 1W LED Epistar, 100Lm, Warm White Voltage: 3V-3.4V, 350 mA"
Changed lines of the file:
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@@
 <part name="G1" library="battery" deviceset="SL-160AA/PT" device="" value="18650"/>
 <part name="LED1" library="display-hp" deviceset="HLMP6" device="" value="1W"/>
-<part name="R3" library="resistor" deviceset="R-EU_" device="0204/2V" value="2R"/>
+<part name="R3" library="resistor" deviceset="R-EU_" device="0204/2V" value="5R"/>
 <part name="GND5" library="supply1" deviceset="GND" device=""/>
 <part name="Q2" library="transistor-power" deviceset="IRF4905" device="" value="AP3310G"/>
@@
 <sheet>
 <plain>
+<text x="60.96" y="30.48" size="1.778" layer="97">2. 1W LED
+    Epistar, 100Lm, Warm White
+    Voltage: 3V-3.4V, 350 mA</text>
+<text x="60.96" y="40.64" size="1.778" layer="97">1. R3 can be replaced by driver
+    NSI50350AST3G  350mA.</text>
 </plain>
 <instances>
